File: sertest-ng.kicad_pcb (KiCad board)
At the start: 4 copper layers, 50 x 160 mm, 152 parts, among them J101 USB, J102 SWD, J201 Debug, J202 RS-232, J203 RS-485/422, J301 USB, J401 CAN, J402 CAN, SW101 Reset, SW401 Term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

Commit message: Add BOOT0 support
Signed-off-by: Benedikt Spranger <b.spranger@linutronix.de>
Parts:
- added JP103: BOOT0, Jumper:SolderJumper-2_P1.3mm_Open_Pad1.0x1.5mm, F.Cu at (129.0, 126.2)
- added R115: 10k, Resistor_SMD:R_0402_1005Metric, F.Cu at (132.5, 125.8)
Routing:
- net /FDCAN1_RX: track 48.8 -> 53.1 mm, vias 2 -> 3
- net +3V3: track 312.1 -> 314.8 mm
- net Net-(U201-R2IN): track 39.4 -> 38.8 mm

Commit message: Add second EEPROM
Signed-off-by: Benedikt Spranger <b.spranger@linutronix.de>
Parts:
- added R116: 1k, Resistor_SMD:R_0402_1005Metric, F.Cu at (138.0, 124.5)
- added U106: M24C64-RMN, Package_SO:SOIC-8_3.9x4.9mm_P1.27mm, F.Cu at (135.2, 117.2)
- moved U101 18.8 mm to (118.8, 126.2), turned to 0 degrees
- moved R101 13.3 mm to (124.8, 123.2), turned to 90 degrees
- moved JP101 10.4 mm to (124.8, 126.2), turned to 90 degrees
Connections:
- net /ISC2_SCL renamed /I2C2_SCL
- U103 pad 44: unconnected-(U103-PA10-Pad44) -> /WP
Routing:
- net /I2C2_SCL: track 9.92 -> 32.8 mm, vias 2 -> 3
- net /I2C2_SDA: track 14.6 -> 36.9 mm, vias 2 -> 3
- net /WP: track 0.00 -> 20.1 mm, vias 0 -> 3
- net Net-(JP101-B): track 11.9 -> 5.37 mm, vias 2 -> 0
- net +3V3: track 314.8 -> 320.0 mm
- net /EN: track 91.0 -> 92.4 mm

Commit message: Bump to v0.2
Signed-off-by: Benedikt Spranger <b.spranger@linutronix.de>
Other:
- board text added: "serttest-NG v0.2 Benedikt Spranger"
- board text removed: "serttest-NG v0.1 Benedikt Spranger"
Changed lines of the file:
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@@
 	(title_block
 		(title "Serial Tester")
-		(date "09.12.2025")
-		(rev "0.1")
+		(date "2026-03-22")
+		(rev "0.2")
 		(company "Eurovibes / Benedikt Spranger")
 		(comment 1 "SPDX-License-Identifier: CERN-OHL-S-2.0")
@@
 		(layer "Edge.Cuts")
 	)
-	(gr_text "serttest-NG v0.1\nBenedikt Spranger"
+	(gr_text "serttest-NG v0.2\nBenedikt Spranger"
 		(at 100 179 0)
 		(layer "F.Cu")
