File: usbserial.kicad_sch (KiCad schematic)
At the start: 13 parts, among them J301 USB, U301 XC6206P332MR, U302 CH340N, U303 USBLC6-2SC6

Commit message: Replace JLCPCB part to fit footprint
Signed-off-by: Benedikt Spranger <b.spranger@linutronix.de>
Parts:
- C301, C302: Long Description 1uF 25V X5R ±10% 0402 Multilayer Ceramic Capacitors MLCC - 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 -> 1uF 50V X5R ±10% 0603 Multilayer Ceramic Capacitors MLCC - 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; MP CL05A105KA5NQNC -> CL10A105KB8NNNC; SupplLink https://jlcpcb.com/partdetail/53938-CL05A105KA5NQNC/C52923 -> https://jlcpcb.com/partdetail/16531-CL10A105KB8NNNC/C15849; lcsc# C52923 -> C15849
Changed lines of the file:
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@@
 			)
 		)
-		(property "Long Description" "1uF 25V X5R ±10% 0402 Multilayer Ceramic Capacitors MLCC - SMD/SMT ROHS"
+		(property "Long Description" "1uF 50V X5R ±10% 0603 Multilayer Ceramic Capacitors MLCC - SMD/SMT ROHS"
 			(at 160.02 57.15 0)
 			(effects
@@
 			)
 		)
-		(property "MP" "CL05A105KA5NQNC"
+		(property "MP" "CL10A105KB8NNNC"
 			(at 160.02 57.15 0)
 			(effects
@@
 			)
 		)
-		(property "SupplLink" "https://jlcpcb.com/partdetail/53938-CL05A105KA5NQNC/C52923"
+		(property "SupplLink" "https://jlcpcb.com/partdetail/16531-CL10A105KB8NNNC/C15849"
 			(at 160.02 57.15 0)
 			(effects
@@
 			)
 		)
-		(property "lcsc#" "C52923"
+		(property "lcsc#" "C15849"
 			(at 160.02 57.15 0)
 			(effects
@@
 			)
 		)
-		(property "Long Description" "1uF 25V X5R ±10% 0402 Multilayer Ceramic Capacitors MLCC - SMD/SMT ROHS"
+		(property "Long Description" "1uF 50V X5R ±10% 0603 Multilayer Ceramic Capacitors MLCC - SMD/SMT ROHS"
 			(at 134.62 57.15 0)
 			(effects
@@
 			)
 		)
-		(property "MP" "CL05A105KA5NQNC"
+		(property "MP" "CL10A105KB8NNNC"
 			(at 134.62 57.15 0)
 			(effects
@@
 			)
 		)
-		(property "SupplLink" "https://jlcpcb.com/partdetail/53938-CL05A105KA5NQNC/C52923"
+		(property "SupplLink" "https://jlcpcb.com/partdetail/16531-CL10A105KB8NNNC/C15849"
 			(at 134.62 57.15 0)
 			(effects
@@
 			)
 		)
-		(property "lcsc#" "C52923"
+		(property "lcsc#" "C15849"
 			(at 134.62 57.15 0)
 			(effects

Commit message: Add USB termination resistors
Signed-off-by: Benedikt Spranger <b.spranger@linutronix.de>
Parts:
- renumbered R302 to R301, R303 to R302, R301 to R303, U303 to U301, U301 to U302, U302 to U303
Changed lines of the file:
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@@
 		(on_board yes)
 		(dnp no)
-		(property "Reference" "R302"
+		(property "Reference" "R301"
 			(at 110.49 73.914 90)
 			(effects
@@
 			(project "sertest-ng"
 				(path "/9a3cad5d-0a7b-485e-a592-d3e508a0fc7b/2df5aafc-bbfd-4dd1-a656-1eb9fd26d032"
-					(reference "R302")
+					(reference "R301")
 					(unit 1)
 				)
@@
 		(on_board yes)
 		(dnp no)
-		(property "Reference" "U303"
+		(property "Reference" "U301"
 			(at 132.334 80.264 0)
 			(effects
@@
 			(project "sertest-ng"
 				(path "/9a3cad5d-0a7b-485e-a592-d3e508a0fc7b/2df5aafc-bbfd-4dd1-a656-1eb9fd26d032"
-					(reference "U303")
+					(reference "U301")
 					(unit 1)
 				)
@@
 		(on_board yes)
 		(dnp no)
-		(property "Reference" "R303"
+		(property "Reference" "R302"
 			(at 110.49 81.026 90)
 			(effects
@@
 			(project "sertest-ng"
 				(path "/9a3cad5d-0a7b-485e-a592-d3e508a0fc7b/2df5aafc-bbfd-4dd1-a656-1eb9fd26d032"
-					(reference "R303")
+					(reference "R302")
 					(unit 1)
 				)
@@
 		(dnp no)
 		(fields_autoplaced yes)
-		(property "Reference" "R301"
+		(property "Reference" "R303"
 			(at 190.5 66.0399 0)
 			(effects
@@
 			(project "sertest-ng"
 				(path "/9a3cad5d-0a7b-485e-a592-d3e508a0fc7b/2df5aafc-bbfd-4dd1-a656-1eb9fd26d032"
-					(reference "R301")
+					(reference "R303")
 					(unit 1)
 				)
@@
 		(dnp no)
 		(fields_autoplaced yes)
-		(property "Reference" "U302"
+		(property "Reference" "U303"
 			(at 209.2041 73.66 0)
 			(effects
@@
 			(project "sertest-ng"
 				(path "/9a3cad5d-0a7b-485e-a592-d3e508a0fc7b/2df5aafc-bbfd-4dd1-a656-1eb9fd26d032"
-					(reference "U302")
+					(reference "U303")
 					(unit 1)
 				)
@@
 		(dnp no)
 		(fields_autoplaced yes)
-		(property "Reference" "U301"
+		(property "Reference" "U302"
 			(at 149.86 44.45 0)
 			(effects
@@
 			(project "sertest-ng"
 				(path "/9a3cad5d-0a7b-485e-a592-d3e508a0fc7b/2df5aafc-bbfd-4dd1-a656-1eb9fd26d032"
-					(reference "U301")
-					(unit 1)
-				)
+					(reference "U302")
+					(unit 1)
+				)
